File: hardware/board_g0/line_sensor.brd (EAGLE design)
At the start: 104 x 52.7 mm, 68 parts, among them IC1 STM32F051K4U, J1 XF2L-0535-1, J5 XF2L-0535-1, Q1 BSS123

Commit message: new hw, firmware for stm32g031
Parts:
- removed IC1: STM32F051K4U, micro-stm_v3:UFQFPN32
- added U$14: STM32G031K8U6, my_library:UFQFPN32
Connections:
- removed net BOOT: J3.3, R25.2
- removed net SWCLK: J3.2
- removed net VDDA: IC1.5
- new net SWCLK/BOOT: J3.2, J3.3, R25.2, U$14.25
- net +3V3: now also U$14.4; no longer IC1.1, IC1.17
- net ADC0: now also U$14.7
- net ADC1: now also U$14.8
- net ADC2: now also U$14.9
- net ADC3: now also U$14.10
- net ADC4: now also U$14.11
- net ADC5: now also U$14.12
- net ADC6: now also U$14.13
- net ADC7: now also U$14.14
- net ADC8: now also U$14.15
- net ADC9: now also U$14.16
- net ADR: now also U$14.26
- net GND: now also U$14.5, U$14.VSS; no longer IC1.VSS
- net LED: now also U$14.18
- net LED_CONTROL: now also U$14.17
- net RESET: now also U$14.6
- net SCL: now also U$14.32
- net SDA: now also U$14.31
- net SWDIO: now also U$14.24
- net UART_RX: now also U$14.21
- net UART_TX: now also U$14.19
Routing:
- net +3V3: track 182.6 -> 169.0 mm, vias 7 -> 6
- net SWCLK/BOOT: track 0.00 -> 13.0 mm
- net BOOT: track 9.64 -> 0.00 mm
- net SWCLK: track 7.65 -> 0.00 mm
- net RESET: track 44.6 -> 50.1 mm, vias 3 -> 2
- net GND: track 222.7 -> 228.1 mm, vias 71 -> 74
- net SDA: track 22.8 -> 25.6 mm
- net ADC2: track 34.9 -> 32.4 mm
- net ADR: track 2.01 -> 4.38 mm
- net ADC3: track 21.2 -> 23.3 mm
- net ADC4: track 9.67 -> 11.4 mm
- net ADC5: track 22.5 -> 24.2 mm
- net UART_TX: track 9.07 -> 10.7 mm
- net SCL: track 22.3 -> 24.0 mm
- net LED: track 8.28 -> 9.71 mm
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