File: hardware/board_g0/line_sensor.sch (EAGLE design)
At the start: 68 parts, among them IC1 STM32F051K4U, J1 XF2L-0535-1, J5 XF2L-0535-1, Q1 BSS123

Commit message: new hw, firmware for stm32g031
Parts:
- removed IC1: STM32F051K4U, micro-stm_v3:STM32F051K4U
- added U$14: STM32G031K8U6, my_library:STM32G031K8U6
Connections:
- removed net BOOT: J3.3, R25.2
- removed net SWCLK: J3.2
- new net SWCLK/BOOT: J3.2, J3.3, R25.2, U$14.PA14/BOOT0
- net +3V3: now also U$14.VDD/VDDA; no longer IC1PWR.VDD@1, IC1PWR.VDD@2
- net ADC0: now also U$14.PA0
- net ADC1: now also U$14.PA1
- net ADC2: now also U$14.PA2
- net ADC3: now also U$14.PA3
- net ADC4: now also U$14.PA4
- net ADC5: now also U$14.PA5
- net ADC6: now also U$14.PA6
- net ADC7: now also U$14.PA7
- net ADC8: now also U$14.PB0
- net ADC9: now also U$14.PB1
- net ADR: now also U$14.PA15
- net GND: now also U$14.VSS-PAD, U$14.VSS/VSSA; no longer IC1PWR.VSS@1
- net LED: now also U$14.PA8
- net LED_CONTROL: now also U$14.PB2
- net RESET: now also U$14.NRST/PF2
- net SCL: now also U$14.PB8
- net SDA: now also U$14.PB7
- net SWDIO: now also U$14.PA13
- net UART_RX: now also U$14.PA10
- net UART_TX: now also U$14.PA9
