File: hardware/board_g0_slim/line_sensor.brd (EAGLE design)
At the start: 104 x 52.7 mm, 70 parts, among them J1 XF2L-0535-1, J5 XF2L-0535-1, Q1 BSS123

Commit message: working firmware v1
Parts:
- removed H1, H2, H3, H4, H5, H6: MOUNT-HOLE3.0, holes:3,0
- removed J3: (no value), SparkFun-Connectors:2X4
- removed J4: (no value), SparkFun-Connectors:1X05
- removed J5: XF2L-0535-1, con-omron:XF2L-0535-1
- added U$15: DEBUG_CON, my_library:HEADER_4X2_1.27
- moved U$13 4.12 mm to (99.0, 40.0)
- moved D2 3.00 mm to (86.0, 42.5)
- moved U$2 3.00 mm to (89.0, 42.5)
- moved D10 2.55 mm to (12.5, 39.5)
- moved D3 2.50 mm to (76.0, 44.8)
- moved U$10 2.50 mm to (9.50, 39.8)
- moved U$12 2.50 mm to (9.50, 40.0)
- moved D1 2.46 mm to (96.0, 40.0)
- moved D9 2.06 mm to (22.0, 43.0)
- moved U$9 2.06 mm to (19.0, 43.0)
- moved D7 2.00 mm to (42.0, 46.0)
- moved D8 2.00 mm to (32.0, 44.8)
- moved U$1 2.00 mm to (99.0, 40.0)
- moved U$3 2.00 mm to (79.0, 44.8)
- moved U$7 2.00 mm to (39.0, 46.0)
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Connections:
- net +3V3: now also U$15.P$1; no longer J3.1, J4.5, J5.1
- net GND: now also U$15.P$4; no longer J3.7, J4.1, J5.5
- net RESET: now also U$15.P$5; no longer J3.5, J4.2, J5.4
- net SCL: no longer J4.4, J5.2
- net SDA: no longer J4.3, J5.3
- net SWCLK/BOOT: now also U$15.P$6, U$15.P$7; no longer J3.2, J3.3
- net SWDIO: now also U$15.P$8; no longer J3.4
- net UART_RX: now also U$15.P$3; no longer J3.6
- net UART_TX: now also U$15.P$2; no longer J3.8
Routing:
- net ADC9: track 53.9 -> 2.56 mm, vias 1 -> 0
- net GND: track 174.1 -> 136.4 mm, vias 65 -> 17
- net N$11: track 58.9 -> 29.4 mm
- net +3V3: track 169.0 -> 160.9 mm
- net SWCLK/BOOT: track 13.0 -> 6.90 mm
- net RESET: track 50.1 -> 44.5 mm
- net SCL: track 24.0 -> 18.4 mm
- net ADC8: track 46.8 -> 42.4 mm, vias 1 -> 0
- net SDA: track 25.6 -> 21.5 mm
- net ADC1: track 48.1 -> 45.1 mm
- net UART_TX: track 10.7 -> 7.94 mm
- net N$10: track 2.55 -> 0.00 mm
- net ADC6: track 29.6 -> 27.2 mm
- net N$9: track 2.30 -> 0.00 mm
- net N$8: track 2.30 -> 0.00 mm
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Other:
- board size 104 x 52.7 mm -> 100 x 31.3 mm
- board text added: "r = 150.00"
- board text removed: "r = 150"

Commit message: demo codes, cleaned up
Parts:
- removed C4: 10n, rcl:C0805K
- removed U$11: FIDUCIAL, borkedlabs-misc:FIDUCIAL_1MM
- removed U$15: DEBUG_CON, my_library:HEADER_4X2_1.27
- added D12, D13: WHITE, SparkFun-LED:LED-1206
- added J3: (no value), SparkFun-Connectors:1X04_LOCK
- added R27, R28: 330, rcl:M0805
- moved R21 23.5 mm to (40.6, 45.9), turned to 90 degrees
- moved Q1 20.1 mm to (43.7, 45.6), turned to 270 degrees
- moved R23 7.44 mm to (60.9, 36.0), flipped to the bottom, turned to 270 degrees
- moved J1 6.08 mm to (55.0, 27.0)
- moved J2 6.08 mm to (50.0, 32.0)
- moved U$14 6.08 mm to (55.0, 41.0), turned to 225 degrees
- moved SJ1 6.06 mm to (54.9, 38.0)
- moved C2 5.70 mm to (63.4, 33.8)
- moved R26 5.61 mm to (50.2, 49.5), turned to 180 degrees
- moved R25 5.57 mm to (50.6, 35.1), turned to 0 degrees
- moved R22 5.12 mm to (58.8, 36.0), flipped to the bottom, turned to 270 degrees
- moved D11 5.02 mm to (55.0, 49.4)
- moved H8 4.00 mm to (14.0, 28.0)
- moved R24 3.34 mm to (63.5, 37.9), turned to 0 degrees
- moved H7 3.16 mm to (96.0, 28.0)
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Connections:
- removed net SWCLK/BOOT: R25.2, U$14.25, U$15.P$6, U$15.P$7
- new net N$13: D12.A, R27.1
- new net N$14: D13.A, R28.1
- new net SWCLK: J3.3, R25.2, U$14.25
- net +3V3: now also R27.2, R28.2; no longer U$15.P$1
- net GND: now also J3.1; no longer C4.2, U$15.P$4
- net N$11: now also D12.C, D13.C
- net RESET: now also J3.2; no longer C4.1, U$15.P$5
- net SWDIO: now also J3.4; no longer U$15.P$8
- net UART_RX: no longer U$15.P$3
- net UART_TX: no longer U$15.P$2
Routing:
- net N$11: track 29.4 -> 132.6 mm, vias 0 -> 1
- net GND: track 136.4 -> 193.5 mm, vias 17 -> 27
- net ADC9: track 2.56 -> 49.3 mm, vias 0 -> 1
- net LED: track 9.71 -> 42.0 mm
- net ADC0: track 25.4 -> 54.6 mm, vias 0 -> 1
- net ADC5: track 25.5 -> 11.9 mm
- net LED_CONTROL: track 17.7 -> 29.4 mm
- net SWCLK: track 0.00 -> 11.4 mm
- net ADC7: track 35.9 -> 25.8 mm
- net ADC4: track 12.2 -> 22.0 mm
- net UART_RX: track 9.60 -> 0.00 mm
- net ADC3: track 20.9 -> 29.9 mm
- net +3V3: track 160.9 -> 152.3 mm, vias 6 -> 2
- net RESET: track 44.5 -> 36.2 mm, vias 2 -> 1
- net UART_TX: track 7.94 -> 0.00 mm
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- added copper zone on layer 1, net GND
- added copper zone on layer 16, net GND
Other:
- board size 100 x 31.3 mm -> 108 x 27 mm
- board text removed: "BOOT"
- board text removed: "UART_RX"
- board text removed: "UART_TX"
