File: hardware/board_g0_slim/line_sensor.sch (EAGLE design)
At the start: 70 parts, among them J1 XF2L-0535-1, J5 XF2L-0535-1, Q1 BSS123

Commit message: working firmware v1
Parts:
- removed H1, H2, H3, H4, H5, H6: MOUNT-HOLE3.0, holes:MOUNT-HOLE3.0
- removed J3: (no value), SparkFun-Connectors:CONN_04X2
- removed J4: (no value), SparkFun-Connectors:CONN_05
- removed J5: XF2L-0535-1, con-omron:XF2L-0535-1
- added U$15: DEBUG_CON, my_library:DEBUG_CON
Connections:
- net +3V3: now also U$15.VCC; no longer J3.1, J4.5, J5-1.MSV
- net GND: now also U$15.GND; no longer J3.7, J4.1, J5-5.MS
- net RESET: now also U$15.RESET; no longer J3.5, J4.2, J5-4.MS
- net SCL: no longer J4.4, J5-2.MS
- net SDA: no longer J4.3, J5-3.MS
- net SWCLK/BOOT: now also U$15.BOOT, U$15.SWCLK; no longer J3.2, J3.3
- net SWDIO: now also U$15.SWDIO; no longer J3.4
- net UART_RX: now also U$15.RX; no longer J3.6
- net UART_TX: now also U$15.TX; no longer J3.8

Commit message: demo codes, cleaned up
Parts:
- removed C4: 10n, rcl:C-EUC0805K
- removed U$11: FIDUCIAL, borkedlabs-misc:FIDUCIAL
- removed U$15: DEBUG_CON, my_library:DEBUG_CON
- added D12, D13: WHITE, SparkFun-LED:LED-WHITE1206
- added J3: (no value), SparkFun-Connectors:CONN_04LOCK
- added R27, R28: 330, rcl:R-EU_M0805
Connections:
- removed net SWCLK/BOOT: R25.2, U$14.PA14/BOOT0, U$15.BOOT, U$15.SWCLK
- new net N$13: D12.A, R27.1
- new net N$14: D13.A, R28.1
- new net SWCLK: J3.3, R25.2, U$14.PA14/BOOT0
- net +3V3: now also R27.2, R28.2; no longer U$15.VCC
- net GND: now also J3.1; no longer C4.2, U$15.GND
- net N$11: now also D12.C, D13.C
- net RESET: now also J3.2; no longer C4.1, U$15.RESET
- net SWDIO: now also J3.4; no longer U$15.SWDIO
- net UART_RX: no longer U$15.RX
- net UART_TX: no longer U$15.TX
Other:
- moved on the sheet: C1, C2, C3, D1, D10, D2, D3, D4, D5, D6, D7, D8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
