File: hardware/board_v2/line_sensor.brd (EAGLE design)
At the start: 108 x 27 mm, 64 parts, among them J1 XF2L-0535-1, Q1 BSS123

Commit message: updated v2 firmware
Parts:
- added R29, R30, R31, R32: 4k7, rcl:M0805
- added R33, R34, R35, R36: 22, rcl:M0805
- added SJ2: (no value), jumper:SJ
- added U$11, U$15, U$16, U$17, U$18, U$19, U$20, U$21: LED_5MM_AXIAL, my_library:LED_5MM_AXIAL
- moved J3 4.00 mm to (46.3, 27.1)
- moved R5 2.40 mm to (63.2, 44.3), turned to 180 degrees
- moved R24 1.26 mm to (63.2, 36.7)
- moved R6 0.96 mm to (48.9, 42.6)
- moved R16 0.30 mm to (51.0, 42.6)
- renumbered Q1 to Q1PMV37ENEA
Connections:
- new net ADC10: R32.1, U$14.17, U$21.P$2
- new net ADC15: R30.1, U$14.22, U$17.P$2
- new net ADC16: R29.1, U$14.23, U$15.P$2
- new net ADC17: R31.1, SJ2.1, U$19.P$2
- new net LED_SW: D1.C, D10.C, D12.C, D13.C, D2.C, D3.C, D4.C, D5.C, D6.C, D7.C, D8.C, D9.C, Q1PMV37ENEA.3, U$11.P$2, U$16.P$2, U$18.P$2, U$20.P$2
- new net N$19: R34.1, U$16.P$1
- new net N$20: R35.1, U$18.P$1
- new net N$21: R36.1, U$20.P$1
- net +3V3: now also R29.2, R30.2, R31.2, R32.2, R33.2, R34.2, R35.2, R36.2
- net GND: now also U$15.P$1, U$17.P$1, U$19.P$1, U$21.P$1
- net LED_CONTROL: now also U$14.20; no longer U$14.17
- net N$11: now also R33.1, U$11.P$1; no longer D1.C, D10.C, D12.C, D13.C, D2.C, D3.C, D4.C, D5.C, D6.C, D7.C, D8.C, D9.C, Q1PMV37ENEA.3
- net SWDIO: now also SJ2.2
Routing:
- net LED_SW: track 0.00 -> 232.6 mm, vias 0 -> 4
- net N$11: track 132.6 -> 4.09 mm, vias 1 -> 0
- net GND: track 193.5 -> 252.5 mm, vias 27 -> 31
- net ADC10: track 0.00 -> 58.0 mm, vias 0 -> 3
- net SWDIO: track 8.88 -> 49.9 mm
- net ADC16: track 0.00 -> 31.1 mm
- net +3V3: track 152.3 -> 166.6 mm
- net ADC15: track 0.00 -> 10.3 mm, vias 0 -> 1
- net ADC17: track 0.00 -> 6.52 mm
- net N$19: track 0.00 -> 4.99 mm
- net N$21: track 0.00 -> 4.67 mm
- net LED_CONTROL: track 29.4 -> 33.9 mm, vias 2 -> 4
- net ADC4: track 22.0 -> 19.5 mm
- net N$20: track 0.00 -> 2.35 mm
- net ADR: track 7.25 -> 5.37 mm
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Other:
- outline, holes or cut-outs redrawn
